File: RS485-dry-contact.kicad_pcb (KiCad board)
At the start: 2 copper layers, 40 x 25.4 mm, 21 parts, among them CON1 AVR-ISP-10, IC1 ATMEGA168PA-A, IC2 SP3485EN, P1 CONN_2, P2 CONN_6, P3 CONN_6, P4 CONN_2, P5 CONN_4, P6 CONN_7, U1 7805

Commit message: draft
Parts:
- removed CON1: AVR-ISP-10, PIN_ARRAY_5x2
- added R2: R, SM1206, F.Cu at (145.5, 58.5)
- U1: footprint TO220_VERT -> TO92
- moved D1 88.8 mm to (108.0, 47.6), turned to 90 degrees
- moved P5 49.8 mm to (174.6, 111.8), turned to 180 degrees
- moved C3 28.6 mm to (160.0, 50.8)
- moved C2 21.6 mm to (113.0, 40.6), turned to 180 degrees
- moved R1 20.2 mm to (101.0, 50.8), turned to 90 degrees
- moved P2 11.4 mm to (143.5, 41.3), turned to 90 degrees
- moved P3 10.9 mm to (134.6, 34.9), turned to 0 degrees
- moved IC2 1.27 mm to (123.8, 42.5)
- moved U1 1.27 mm to (116.8, 47.6), turned to 0 degrees
- moved IC1 1.27 mm to (135.3, 43.2)
Connections:
- IC1 pad 15: N-0000012 -> N-000003
- IC1 pad 16: N-0000014 -> N-000009
- IC1 pad 17: N-0000013 -> N-0000011
- IC1 pad 23: N-0000025 -> N-0000010
- IC1 pad 24: N-0000026 -> N-0000015
- IC1 pad 25: N-0000027 -> (no net)
- IC1 pad 26: N-0000028 -> (no net)
- IC1 pad 27: N-0000023 -> (no net)
- IC1 pad 28: N-0000022 -> (no net)
- IC1 pad 29: N-000002 (its old number) -> N-0000014
- P3 pad 1: N-0000025 -> N-000003
- P3 pad 2: N-0000026 -> N-000009
- P3 pad 3: N-0000027 -> N-0000011
- P3 pad 4: N-0000028 -> N-0000010
- P3 pad 5: N-0000023 -> N-0000015
- P3 pad 6: N-0000022 -> N-0000014
Routing:
- net N-000004: track 0.00 -> 22.8 mm
- net GND: track 0.00 -> 15.5 mm
- net N-0000031: track 0.00 -> 13.0 mm
- net N-000002: track 0.00 -> 8.78 mm
- net VCC: track 0.00 -> 6.40 mm
- net N-0000033: track 0.00 -> 5.71 mm
- net N-0000032: track 0.00 -> 5.71 mm
- net N-0000020: track 0.00 -> 4.53 mm
- net N-0000019: track 0.00 -> 4.34 mm
- net N-000007: track 3.63 -> 0.00 mm
- net N-000006: track 3.52 -> 0.00 mm
- net N-000005: track 0.00 -> 1.91 mm

Commit message: draft
Parts:
- removed C6: CP1, CP8
- removed P5: CONN_4, bornier4
- added X1: CRYSTAL, crystal_FA238-TSX3225, B.Cu at (116.2, 85.1)
- C1: footprint CP10 -> c_tant_D
- C7, C8, R2: moved to B.Cu
- D1: footprint LED-3MM -> LED-1206
- R1: moved to F.Cu
- moved C1 75.5 mm to (131.4, 77.5), turned to 180 degrees
- moved C2 47.8 mm to (128.9, 85.7), turned to 90 degrees
- moved P4 46.6 mm to (141.0, 79.4), turned to 90 degrees
- moved P1 42.0 mm to (108.6, 79.4), turned to 270 degrees
- moved C3 40.7 mm to (137.2, 84.5), turned to 90 degrees
- moved U1 39.5 mm to (132.7, 83.8), turned to 270 degrees
- moved P3 38.4 mm to (121.9, 71.1)
- moved IC1 38.4 mm to (122.6, 79.4)
- moved IC2 37.6 mm to (134.0, 78.7), turned to 90 degrees
- moved R1 37.0 mm to (124.5, 79.4), turned to 270 degrees
- moved P6 36.2 mm to (122.6, 90.8)
- moved D2 35.0 mm to (114.3, 78.1), turned to 270 degrees
- moved D1 31.9 mm to (120.7, 76.8), turned to 180 degrees
- moved C5 31.1 mm to (118.7, 74.3), turned to 180 degrees
- moved P2 30.5 mm to (137.2, 71.1), turned to 180 degrees
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Connections:
- IC1 pad 1: N-0000018 (its old number) -> (no net)
- IC1 pad 10: N-0000020 (its old number) -> (no net)
- IC1 pad 11: N-0000016 -> (no net)
- IC1 pad 12: N-0000019 -> (no net)
- IC1 pad 13: N-000007 (its old number) -> (no net)
- IC1 pad 14: N-000006 (its old number) -> (no net)
- IC1 pad 27: (no net) -> N-0000014
- IC1 pad 28: (no net) -> N-0000015
- IC1 pad 9: N-000001 -> N-0000016
- IC2 pad 2: N-000006 (its old number) -> N-0000015
- IC2 pad 3: N-000007 (its old number) -> N-0000014
- P6 pad 1: N-0000018 (its old number) -> N-0000016
Routing:
- net GND: track 15.5 -> 183.2 mm
- net (no net): track 0.00 -> 88.7 mm
- net VCC: track 6.40 -> 58.5 mm
- net N-0000031: track 13.0 -> 34.6 mm
- net N-0000016: track 0.00 -> 16.2 mm, vias 0 -> 1
- net N-0000012: track 0.00 -> 15.9 mm
- net N-000006: track 22.8 -> 11.0 mm
- net N-0000034: track 0.00 -> 10.9 mm
- net N-0000035: track 0.00 -> 9.74 mm
- net N-0000020: track 0.00 -> 8.07 mm
- net N-0000018: track 0.00 -> 6.83 mm
- net N-000009: track 0.00 -> 5.60 mm
- net N-0000020 (its old number): track 4.53 -> 0.00 mm
- net N-0000019: track 4.34 -> 0.00 mm
- net N-0000010: track 0.00 -> 4.08 mm
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Other:
- board size 40 x 25.4 mm -> 40.6 x 61.6 mm

Commit message: Rev 1.0
Parts:
- removed P6: CONN_7, bornier6
- added D3: LED, LED-1206, F.Cu at (128.9, 85.7)
- added D4: LED, LED-1206, F.Cu at (131.4, 74.3)
- added D5: LED, LED-1206, F.Cu at (123.2, 84.5)
- added K1: CONN_3, bornier3, F.Cu at (114.9, 90.8)
- added P5: CONN_4, bornier4, F.Cu at (132.7, 90.8)
- added R3: R, SM1206, F.Cu at (124.5, 87.0)
- added R4: R, SM1206, F.Cu at (126.4, 74.3)
- added R5: R, SM1206, F.Cu at (118.7, 87.0)
- moved C1 0.64 mm to (132.1, 77.5)
Connections:
- IC1 pad 1: (no net) -> N-0000015
Routing:
- net (no net): track 88.7 -> 0.00 mm
- net GND: track 183.2 -> 210.1 mm, vias 0 -> 2
- net N-0000014: track 3.45 -> 13.5 mm, vias 0 -> 1
- net N-0000035: track 34.6 -> 39.6 mm
- net VCC: track 58.5 -> 62.9 mm, vias 0 -> 2
- net N-0000015: track 0.00 -> 3.59 mm, vias 0 -> 1
- net N-0000016: track 0.00 -> 3.39 mm
- net N-0000018: track 11.0 -> 14.4 mm, vias 0 -> 1
- net N-0000013: track 0.00 -> 2.80 mm
- net N-000004: track 16.2 -> 18.6 mm
- net N-0000012: track 0.00 -> 2.01 mm
- added copper zone on B.Cu, net GND
- added copper zone on F.Cu, net GND
Other:
- board size 40.6 x 61.6 mm -> 40 x 25.4 mm

Commit message: Rev 1.1
Parts:
- ?: renamed from P4; value CONN_2 -> B 485 A
- ?: renamed from D4; value LED -> TxD
- ?: renamed from D5; value LED -> Status
- ?: renamed from P1; value CONN_2 -> PSupply
- ?: renamed from P2; value CONN_6 -> (none)
- ?: renamed from P3; value CONN_6 -> (none)
- ?: renamed from U1; value 7805 -> (none)
- ?: renamed from D1; value LED -> Power
- ?: renamed from D3; value LED -> RxD
- ?: renamed from P5; value CONN_4 -> (none)
- ?: renamed from K1; value CONN_3 -> (none)
- C1: value CP1 -> (none)
- C2, C3, C4, C5, C7, C8: value C -> (none)
- D2: value BRIDGE -> (none)
- IC1: value ATMEGA168PA-A -> (none)
- IC2: value SP3485EN -> (none)
- R1, R2, R4, R5: value R -> (none)
- R3: value R -> (none); moved to B.Cu
- X1: value CRYSTAL -> (none)
- moved R3 16.5 mm to (141.0, 86.4), turned to 90 degrees
- moved R5 3.86 mm to (118.1, 83.2), turned to 90 degrees
- moved ? 1.27 mm to (128.9, 84.5)
Routing:
- net GND: track 210.1 -> 185.1 mm, vias 2 -> 3
- net N-000004: track 18.6 -> 42.0 mm
- net N-0000013: track 2.80 -> 13.2 mm, vias 0 -> 1
- net N-0000035: track 39.6 -> 47.9 mm, vias 0 -> 1
- net N-0000014: track 13.5 -> 12.2 mm
- net N-0000016: track 3.39 -> 4.18 mm
- net N-0000038: track 11.3 -> 11.9 mm
Other:
- board text added: "by BG rev 1.1"
