File: RS485-dry-contact.sch (KiCad schematic (older format))
At the start: 22 parts, among them CON1 AVR-ISP-10, IC1 ATMEGA168PA-A, IC2 SP3485EN, P1 CONN_2, P2 CONN_6, P3 CONN_6, P4 CONN_2, P5 CONN_4, P6 CONN_7, U1 7805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

Commit message: draft
Parts:
- removed CON1: AVR-ISP-10, AVR-ISP-10, symbol AVR-ISP-10
- added R2: R, ~, symbol R
Connections:
- wire segments 116 -> 113
- no-connect marks 6 -> 5
Changed lines of the file:
@@
 $EndComp
 $Comp
-L AVR-ISP-10 CON1
-U 1 1 5529019E
-P 8800 2900
-F 0 "CON1" H 8630 3230 50  0000 C CNN
-F 1 "AVR-ISP-10" H 8460 2570 50  0000 L BNN
-F 2 "AVR-ISP-10" V 8050 2950 50  0001 C CNN
-F 3 "" H 8800 2900 60  0000 C CNN
-	1    8800 2900
-	1    0    0    -1
-$EndComp
-$Comp
-L GND #PWR05
-U 1 1 55290342
-P 9200 3250
-F 0 "#PWR05" H 9200 3250 30  0001 C CNN
-F 1 "GND" H 9200 3180 30  0001 C CNN
-F 2 "" H 9200 3250 60  0000 C CNN
-F 3 "" H 9200 3250 60  0000 C CNN
-	1    9200 3250
-	1    0    0    -1
-$EndComp
-$Comp
-L VCC #PWR06
-U 1 1 552903CC
-P 9200 2400
-F 0 "#PWR06" H 9200 2500 30  0001 C CNN
-F 1 "VCC" H 9200 2500 30  0000 C CNN
-F 2 "" H 9200 2400 60  0000 C CNN
-F 3 "" H 9200 2400 60  0000 C CNN
-	1    9200 2400
-	0    -1   -1   0
-$EndComp
-$Comp
-L VCC #PWR07
+L VCC #PWR05
 U 1 1 55290419
 P 5100 2450
-F 0 "#PWR07" H 5100 2550 30  0001 C CNN
+F 0 "#PWR05" H 5100 2550 30  0001 C CNN
 F 1 "VCC" H 5100 2550 30  0000 C CNN
 F 2 "" H 5100 2450 60  0000 C CNN
@@
 $EndComp
 $Comp
-L GND #PWR08
+L GND #PWR06
 U 1 1 552904E9
 P 5200 5200
-F 0 "#PWR08" H 5200 5200 30  0001 C CNN
+F 0 "#PWR06" H 5200 5200 30  0001 C CNN
 F 1 "GND" H 5200 5130 30  0001 C CNN
 F 2 "" H 5200 5200 60  0000 C CNN
@@
 NoConn ~ 5300 4050
 NoConn ~ 5300 4150
-NoConn ~ 8600 2800
 NoConn ~ 7200 4500
-$Comp
-L CONN_6 P3
-U 1 1 55290DB8
-P 10800 3800
-F 0 "P3" V 10750 3800 60  0000 C CNN
-F 1 "CONN_6" V 10850 3800 60  0000 C CNN
-F 2 "~" H 10800 3800 60  0000 C CNN
-F 3 "~" H 10800 3800 60  0000 C CNN
-	1    10800 3800
-	1    0    0    -1
-$EndComp
 $Comp
 L CONN_2 P4
@@
 $EndComp
 $Comp
-L GND #PWR09
+L GND #PWR07
 U 1 1 55291E59
 P 6200 6600
-F 0 "#PWR09" H 6200 6600 30  0001 C CNN
+F 0 "#PWR07" H 6200 6600 30  0001 C CNN
 F 1 "GND" H 6200 6530 30  0001 C CNN
 F 2 "" H 6200 6600 60  0000 C CNN
@@
 $EndComp
 $Comp
-L VCC #PWR010
+L VCC #PWR08
 U 1 1 55291F2A
 P 6200 5700
-F 0 "#PWR010" H 6200 5800 30  0001 C CNN
+F 0 "#PWR08" H 6200 5800 30  0001 C CNN
 F 1 "VCC" H 6200 5800 30  0000 C CNN
 F 2 "" H 6200 5700 60  0000 C CNN
@@
 $EndComp
 $Comp
-L GND #PWR011
+L GND #PWR09
 U 1 1 55291FA4
 P 8950 5400
-F 0 "#PWR011" H 8950 5400 30  0001 C CNN
+F 0 "#PWR09" H 8950 5400 30  0001 C CNN
 F 1 "GND" H 8950 5330 30  0001 C CNN
 F 2 "" H 8950 5400 60  0000 C CNN
@@
 $EndComp
 $Comp
-L VCC #PWR012
+L VCC #PWR010
 U 1 1 55292029
 P 8950 4400
-F 0 "#PWR012" H 8950 4500 30  0001 C CNN
+F 0 "#PWR010" H 8950 4500 30  0001 C CNN
 F 1 "VCC" H 8950 4500 30  0000 C CNN
 F 2 "" H 8950 4400 60  0000 C CNN
@@
 $EndComp
 $Comp
-L GND #PWR013
+L GND #PWR011
 U 1 1 55292317
 P 10350 3250
-F 0 "#PWR013" H 10350 3250 30  0001 C CNN
+F 0 "#PWR011" H 10350 3250 30  0001 C CNN
 F 1 "GND" H 10350 3180 30  0001 C CNN
 F 2 "" H 10350 3250 60  0000 C CNN
@@
 $EndComp
 $Comp
-L GND #PWR014
+L GND #PWR012
 U 1 1 552937E0
 P 8050 1400
-F 0 "#PWR014" H 8050 1400 30  0001 C CNN
+F 0 "#PWR012" H 8050 1400 30  0001 C CNN
 F 1 "GND" H 8050 1330 30  0001 C CNN
 F 2 "" H 8050 1400 60  0000 C CNN
@@
 $EndComp
 $Comp
-L GND #PWR015
+L GND #PWR013
 U 1 1 552937E6
 P 7450 1400
-F 0 "#PWR015" H 7450 1400 30  0001 C CNN
+F 0 "#PWR013" H 7450 1400 30  0001 C CNN
 F 1 "GND" H 7450 1330 30  0001 C CNN
 F 2 "" H 7450 1400 60  0000 C CNN
@@
 Connection ~ 5200 4900
 Wire Wire Line
-	8600 2700 7550 2700
-Wire Wire Line
-	7550 2700 7550 3000
+	7550 2650 7550 3000
 Wire Wire Line
 	7550 3000 7200 3000
-Wire Wire Line
-	8600 3100 7200 3100
-Wire Wire Line
-	8600 3000 7700 3000
-Wire Wire Line
-	7700 3000 7700 3200
-Wire Wire Line
-	7700 3200 7200 3200
-Wire Wire Line
-	8850 2800 9200 2800
-Wire Wire Line
-	9200 2800 9200 3250
-Wire Wire Line
-	9200 2900 8850 2900
-Wire Wire Line
-	9200 3000 8850 3000
-Connection ~ 9200 2900
-Wire Wire Line
-	9200 3100 8850 3100
-Connection ~ 9200 3000
-Connection ~ 9200 3100
-Wire Wire Line
-	9200 2400 9200 2700
-Wire Wire Line
-	9200 2700 8850 2700
 Connection ~ 5100 2700
 Connection ~ 5200 5000
 Wire Wire Line
-	7200 3550 10450 3550
-Wire Wire Line
-	7200 3650 10450 3650
-Wire Wire Line
-	7200 3750 10450 3750
-Wire Wire Line
-	7200 3850 10450 3850
-Wire Wire Line
-	7200 4050 10450 4050
-Wire Wire Line
-	7200 3950 10450 3950
-Wire Wire Line
-	8600 2900 7850 2900
-Wire Wire Line
-	7850 2900 7850 4150
-Wire Wire Line
-	7850 4150 7200 4150
+	7200 4150 8400 4150
 Wire Wire Line
 	7200 4300 7850 4300
@@
 Connection ~ 10350 2750
 Connection ~ 10350 3150
-Connection ~ 10200 4050
-Connection ~ 10050 3950
-Connection ~ 9900 3850
-Connection ~ 9750 3750
-Connection ~ 9600 3650
-Connection ~ 9450 3550
 Wire Wire Line
 	7450 3300 7200 3300
@@
 NoConn ~ 4350 1750
 $Comp
-L GND #PWR016
+L GND #PWR014
 U 1 1 55295093
 P 4250 2000
-F 0 "#PWR016" H 4250 2000 30  0001 C CNN
+F 0 "#PWR014" H 4250 2000 30  0001 C CNN
 F 1 "GND" H 4250 1930 30  0001 C CNN
 F 2 "" H 4250 2000 60  0000 C CNN
@@
 	4250 2000 4250 1750
 $Comp
-L GND #PWR017
+L GND #PWR015
 U 1 1 55295132
 P 4550 2000
-F 0 "#PWR017" H 4550 2000 30  0001 C CNN
+F 0 "#PWR015" H 4550 2000 30  0001 C CNN
 F 1 "GND" H 4550 1930 30  0001 C CNN
 F 2 "" H 4550 2000 60  0000 C CNN
@@
 	4650 3600 4650 1750
 $Comp
-L GND #PWR018
+L GND #PWR016
 U 1 1 5529525F
 P 4750 2000
-F 0 "#PWR018" H 4750 2000 30  0001 C CNN
+F 0 "#PWR016" H 4750 2000 30  0001 C CNN
 F 1 "GND" H 4750 1930 30  0001 C CNN
 F 2 "" H 4750 2000 60  0000 C CNN
@@
 Wire Wire Line
 	4750 2000 4750 1750
+$Comp
+L CONN_6 P3
+U 1 1 55295FCC
+P 9500 2900
+F 0 "P3" V 9450 2900 60  0000 C CNN
+F 1 "CONN_6" V 9550 2900 60  0000 C CNN
+F 2 "~" H 9500 2900 60  0000 C CNN
+F 3 "~" H 9500 2900 60  0000 C CNN
+	1    9500 2900
+	1    0    0    -1
+$EndComp
+Wire Wire Line
+	7550 2650 9150 2650
+Wire Wire Line
+	7850 2850 9150 2850
+Wire Wire Line
+	7200 3100 7650 3100
+Wire Wire Line
+	7650 3100 7650 2750
+Wire Wire Line
+	7650 2750 9150 2750
+Wire Wire Line
+	7200 3200 7850 3200
+Wire Wire Line
+	7850 3200 7850 2850
+Wire Wire Line
+	7200 3550 8200 3550
+Wire Wire Line
+	8200 3550 8200 2950
+Wire Wire Line
+	8200 2950 9150 2950
+Wire Wire Line
+	9150 3050 8300 3050
+Wire Wire Line
+	8300 3050 8300 3650
+Wire Wire Line
+	8300 3650 7200 3650
+Wire Wire Line
+	8400 4150 8400 3150
+Wire Wire Line
+	8400 3150 9150 3150
+$Comp
+L R R2
+U 1 1 5529650E
+P 9050 3900
+F 0 "R2" V 9130 3900 40  0000 C CNN
+F 1 "R" V 9057 3901 40  0000 C CNN
+F 2 "~" V 8980 3900 30  0000 C CNN
+F 3 "~" H 9050 3900 30  0000 C CNN
+	1    9050 3900
+	0    -1   -1   0
+$EndComp
+Wire Wire Line
+	8800 3900 8400 3900
+Connection ~ 8400 3900
+$Comp
+L VCC #PWR017
+U 1 1 552965A3
+P 9550 3900
+F 0 "#PWR017" H 9550 4000 30  0001 C CNN
+F 1 "VCC" H 9550 4000 30  0000 C CNN
+F 2 "" H 9550 3900 60  0000 C CNN
+F 3 "" H 9550 3900 60  0000 C CNN
+	1    9550 3900
+	0    1    1    0
+$EndComp
+Wire Wire Line
+	9550 3900 9300 3900
 $EndSCHEMATC

Commit message: draft
Parts:
- removed P5: CONN_4, ~, symbol CONN_4
Connections:
- net at IC1.1 ((PCINT19/OC2B/INT1)PD3): no longer P6.1 (P1)
- net at IC1.13 ((PCINT1/OC1A)PB1): no longer IC2.3 (DE)
- net at IC1.14 ((PCINT2/OC1B/~SS~)PB2): no longer IC2.2 (~RE~)
- net at IC1.27 ((PCINT12/SDA/ADC4)PC4): now also IC2.3 (DE)
- net at IC1.28 ((PCINT14/SCL/ADC5)PC5): now also IC2.2 (~RE~)
- net at IC1.9 ((PCINT21/OC0B/T1)PD5): now also P6.1 (P1)
Changed lines of the file:
@@
 Sheet 1 1
 Title ""
-Date "11 apr 2015"
+Date "12 apr 2015"
 Rev ""
 Comp ""
@@
 $EndComp
 $Comp
-L CP1 C6
-U 1 1 55291C6D
-P 6600 6150
-F 0 "C6" H 6650 6250 50  0000 L CNN
-F 1 "CP1" H 6650 6050 50  0000 L CNN
-F 2 "~" H 6600 6150 60  0000 C CNN
-F 3 "~" H 6600 6150 60  0000 C CNN
-	1    6600 6150
-	1    0    0    -1
-$EndComp
-$Comp
 L GND #PWR07
 U 1 1 55291E59
@@
 	1    0    0    -1
 $EndComp
-$Comp
-L CONN_4 P5
-U 1 1 55294242
-P 7000 1600
-F 0 "P5" V 6950 1600 50  0000 C CNN
-F 1 "CONN_4" V 7050 1600 50  0000 C CNN
-F 2 "~" H 7000 1600 60  0000 C CNN
-F 3 "~" H 7000 1600 60  0000 C CNN
-	1    7000 1600
-	0    -1   -1   0
-$EndComp
 Wire Wire Line
 	3700 2150 3700 4650
@@
 Connection ~ 5200 5000
 Wire Wire Line
-	7200 4150 8400 4150
+	8400 4150 7200 4150
 Wire Wire Line
 	7200 4300 7850 4300
@@
 	7750 4400 7200 4400
 Wire Wire Line
-	7200 2800 7400 2800
-Wire Wire Line
-	7400 2800 7400 4950
-Wire Wire Line
-	7400 4950 8550 4950
-Wire Wire Line
-	7200 2900 7250 2900
-Wire Wire Line
-	7250 2900 7250 4850
-Wire Wire Line
-	7250 4850 8550 4850
-Wire Wire Line
 	10450 4800 9350 4800
 Wire Wire Line
@@
 	5800 5950 5800 5850
 Wire Wire Line
-	5800 5850 6600 5850
-Wire Wire Line
-	6600 5850 6600 5950
+	5800 5850 6550 5850
 Wire Wire Line
 	6200 5700 6200 5950
@@
 	5800 6350 5800 6450
 Wire Wire Line
-	5800 6450 6600 6450
-Wire Wire Line
-	6600 6450 6600 6350
+	5800 6450 6550 6450
 Wire Wire Line
 	6200 6350 6200 6600
@@
 	7200 4800 7300 4800
 Wire Wire Line
-	7300 4800 7300 2200
-Wire Wire Line
-	7300 2200 6850 2200
-Wire Wire Line
-	6850 2200 6850 1950
-Wire Wire Line
 	7200 4900 7350 4900
 Wire Wire Line
 	7350 4900 7350 2150
 Wire Wire Line
-	7350 2150 6950 2150
-Wire Wire Line
-	6950 2150 6950 1950
-Wire Wire Line
-	7050 1950 7050 2100
-Wire Wire Line
-	7050 2100 7500 2100
-Wire Wire Line
 	7500 2100 7500 5000
 Wire Wire Line
@@
 Wire Wire Line
 	7200 2700 7250 2700
-Wire Wire Line
-	7250 2700 7250 2050
-Wire Wire Line
-	7250 2050 7150 2050
-Wire Wire Line
-	7150 2050 7150 1950
 $Comp
 L CONN_7 P6
@@
 $EndComp
 Wire Wire Line
-	7200 4600 7450 4600
-Wire Wire Line
-	7450 4600 7450 5400
-Wire Wire Line
-	7450 5400 4150 5400
-Wire Wire Line
-	4150 5400 4150 1750
-Wire Wire Line
 	4450 1750 4450 5350
 Wire Wire Line
@@
 	8300 3650 7200 3650
 Wire Wire Line
-	8400 4150 8400 3150
+	8400 3150 8400 4150
 Wire Wire Line
 	8400 3150 9150 3150
@@
 Wire Wire Line
 	9550 3900 9300 3900
+Wire Wire Line
+	8550 4950 7950 4950
+Wire Wire Line
+	7950 4950 7950 3950
+Wire Wire Line
+	7950 3950 7200 3950
+Wire Wire Line
+	7200 4050 8050 4050
+Wire Wire Line
+	8050 4050 8050 4850
+Wire Wire Line
+	8050 4850 8550 4850
+Wire Wire Line
+	4150 1750 4150 2200
+Wire Wire Line
+	4150 2200 7300 2200
+Wire Wire Line
+	7300 2200 7300 4800
+$Comp
+L CP1 C6
+U 1 1 552A48E4
+P 6550 6150
+F 0 "C6" H 6600 6250 50  0000 L CNN
+F 1 "CP1" H 6600 6050 50  0000 L CNN
+F 2 "~" H 6550 6150 60  0000 C CNN
+F 3 "~" H 6550 6150 60  0000 C CNN
+	1    6550 6150
+	1    0    0    -1
+$EndComp
+Wire Wire Line
+	6550 6450 6550 6350
+Wire Wire Line
+	6550 5850 6550 5950
 $EndSCHEMATC

Commit message: Rev 1.0
Parts:
- removed C6: CP1, ~, symbol CP1
- removed P6: CONN_7, ~, symbol CONN_7
- added D3, D4, D5: LED, ~, symbol LED
- added K1: CONN_3, ~, symbol CONN_3
- added P5: CONN_4, ~, symbol CONN_4
- added R3, R4, R5: R, ~, symbol R
Connections:
- net GND: now also K1.2 (PM), P5.2 (P2), P5.4 (P4), R3.2, R4.2, R5.2
- net at C1.1, C2.2, D2.3 (+)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: now also P5.3 (P3)
- net at IC1.1 ((PCINT19/OC2B/INT1)PD3): now also D5.1 (A)
- net at IC1.2 ((PCINT20/XCK/T0)PD4): now also P5.1 (P1)
- net at IC1.30 ((PCINT16/RXD)PD0), IC2.1 (RO): now also D3.1 (A)
- net at IC1.31 ((PCINT17/TXD)PD1), IC2.4 (DI): now also D4.1 (A)
- net at IC1.9 ((PCINT21/OC0B/T1)PD5): now also K1.1 (P1)
- new net: D3.2 (K), R3.1
- new net: D4.2 (K), R4.1
- new net: D5.2 (K), R5.1
- no-connect marks 5 -> 12
Changed lines of the file:
@@
 Connection ~ 5100 2800
 Wire Wire Line
-	5300 4800 5200 4800
-Wire Wire Line
 	5200 4800 5200 5200
 Wire Wire Line
@@
 Wire Wire Line
 	5200 4900 5300 4900
-Connection ~ 5200 4900
 Wire Wire Line
 	7550 2650 7550 3000
@@
 	7850 4750 8550 4750
 Wire Wire Line
-	8550 5050 7750 5050
+	7750 5050 8550 5050
 Wire Wire Line
 	7750 5050 7750 4400
@@
 	5800 5950 5800 5850
 Wire Wire Line
-	5800 5850 6550 5850
+	5800 5850 6200 5850
 Wire Wire Line
 	6200 5700 6200 5950
@@
 	5800 6350 5800 6450
 Wire Wire Line
-	5800 6450 6550 6450
+	5800 6450 6200 6450
 Wire Wire Line
 	6200 6350 6200 6600
@@
 Connection ~ 10350 3150
 Wire Wire Line
-	7450 3300 7200 3300
-Wire Wire Line
 	7450 1950 7450 3300
 Wire Wire Line
@@
 	8050 3400 7200 3400
 Connection ~ 8050 2200
-Connection ~ 7450 2200
 Wire Wire Line
 	7450 1550 7450 1400
@@
 Wire Wire Line
 	7200 4800 7300 4800
-Wire Wire Line
-	7200 4900 7350 4900
-Wire Wire Line
-	7350 4900 7350 2150
-Wire Wire Line
-	7500 2100 7500 5000
-Wire Wire Line
-	7500 5000 7200 5000
-Wire Wire Line
-	7200 2700 7250 2700
-$Comp
-L CONN_7 P6
-U 1 1 55294EA3
-P 4450 1400
-F 0 "P6" V 4420 1400 60  0000 C CNN
-F 1 "CONN_7" V 4520 1400 60  0000 C CNN
-F 2 "~" H 4450 1400 60  0000 C CNN
-F 3 "~" H 4450 1400 60  0000 C CNN
-	1    4450 1400
-	0    -1   -1   0
-$EndComp
 Wire Wire Line
 	4450 1750 4450 5350
@@
 	7300 2200 7300 4800
 $Comp
-L CP1 C6
-U 1 1 552A48E4
-P 6550 6150
-F 0 "C6" H 6600 6250 50  0000 L CNN
-F 1 "CP1" H 6600 6050 50  0000 L CNN
-F 2 "~" H 6550 6150 60  0000 C CNN
-F 3 "~" H 6550 6150 60  0000 C CNN
-	1    6550 6150
-	1    0    0    -1
-$EndComp
-Wire Wire Line
-	6550 6450 6550 6350
-Wire Wire Line
-	6550 5850 6550 5950
+L CONN_3 K1
+U 1 1 552AB124
+P 4250 1400
+F 0 "K1" V 4200 1400 50  0000 C CNN
+F 1 "CONN_3" V 4300 1400 40  0000 C CNN
+F 2 "~" H 4250 1400 60  0000 C CNN
+F 3 "~" H 4250 1400 60  0000 C CNN
+	1    4250 1400
+	0    -1   -1   0
+$EndComp
+$Comp
+L CONN_4 P5
+U 1 1 552AB135
+P 4600 1400
+F 0 "P5" V 4550 1400 50  0000 C CNN
+F 1 "CONN_4" V 4650 1400 50  0000 C CNN
+F 2 "~" H 4600 1400 60  0000 C CNN
+F 3 "~" H 4600 1400 60  0000 C CNN
+	1    4600 1400
+	0    -1   -1   0
+$EndComp
+NoConn ~ 7200 2700
+NoConn ~ 7200 2800
+NoConn ~ 7200 2900
+NoConn ~ 7200 3750
+NoConn ~ 7200 3850
+NoConn ~ 7200 4900
+NoConn ~ 7200 5000
+$Comp
+L LED D3
+U 1 1 552AB21A
+P 8500 4450
+F 0 "D3" H 8500 4550 50  0000 C CNN
+F 1 "LED" H 8500 4350 50  0000 C CNN
+F 2 "~" H 8500 4450 60  0000 C CNN
+F 3 "~" H 8500 4450 60  0000 C CNN
+	1    8500 4450
+	0    -1   -1   0
+$EndComp
+Wire Wire Line
+	8500 4750 8500 4650
+Connection ~ 8500 4750
+Wire Wire Line
+	8500 4250 8500 4100
+Wire Wire Line
+	8500 4100 8800 4100
+$Comp
+L R R3
+U 1 1 552AB339
+P 9050 4100
+F 0 "R3" V 9130 4100 40  0000 C CNN
+F 1 "R" V 9057 4101 40  0000 C CNN
+F 2 "~" V 8980 4100 30  0000 C CNN
+F 3 "~" H 9050 4100 30  0000 C CNN
+	1    9050 4100
+	0    -1   -1   0
+$EndComp
+Wire Wire Line
+	9300 4100 9550 4100
+$Comp
+L GND #PWR018
+U 1 1 552AB3BD
+P 9550 4100
+F 0 "#PWR018" H 9550 4100 30  0001 C CNN
+F 1 "GND" H 9550 4030 30  0001 C CNN
+F 2 "" H 9550 4100 60  0000 C CNN
+F 3 "" H 9550 4100 60  0000 C CNN
+	1    9550 4100
+	0    -1   -1   0
+$EndComp
+Wire Wire Line
+	7450 3300 7200 3300
+Connection ~ 7450 2200
+$Comp
+L LED D4
+U 1 1 552AB893
+P 8500 5500
+F 0 "D4" H 8500 5600 50  0000 C CNN
+F 1 "LED" H 8500 5400 50  0000 C CNN
+F 2 "~" H 8500 5500 60  0000 C CNN
+F 3 "~" H 8500 5500 60  0000 C CNN
+	1    8500 5500
+	0    1    1    0
+$EndComp
+$Comp
+L R R4
+U 1 1 552AB899
+P 9100 5800
+F 0 "R4" V 9180 5800 40  0000 C CNN
+F 1 "R" V 9107 5801 40  0000 C CNN
+F 2 "~" V 9030 5800 30  0000 C CNN
+F 3 "~" H 9100 5800 30  0000 C CNN
+	1    9100 5800
+	0    -1   -1   0
+$EndComp
+$Comp
+L GND #PWR019
+U 1 1 552AB89F
+P 9550 5800
+F 0 "#PWR019" H 9550 5800 30  0001 C CNN
+F 1 "GND" H 9550 5730 30  0001 C CNN
+F 2 "" H 9550 5800 60  0000 C CNN
+F 3 "" H 9550 5800 60  0000 C CNN
+	1    9550 5800
+	0    -1   -1   0
+$EndComp
+Wire Wire Line
+	9550 5800 9350 5800
+Wire Wire Line
+	8850 5800 8500 5800
+Wire Wire Line
+	8500 5800 8500 5700
+Wire Wire Line
+	8500 5300 8500 5050
+Connection ~ 8500 5050
+Wire Wire Line
+	7200 4600 7650 4600
+Wire Wire Line
+	7650 4600 7650 5300
+$Comp
+L LED D5
+U 1 1 552ABAE8
+P 7650 5500
+F 0 "D5" H 7650 5600 50  0000 C CNN
+F 1 "LED" H 7650 5400 50  0000 C CNN
+F 2 "~" H 7650 5500 60  0000 C CNN
+F 3 "~" H 7650 5500 60  0000 C CNN
+	1    7650 5500
+	0    1    1    0
+$EndComp
+$Comp
+L R R5
+U 1 1 552ABAEE
+P 9100 6000
+F 0 "R5" V 9180 6000 40  0000 C CNN
+F 1 "R" V 9107 6001 40  0000 C CNN
+F 2 "~" V 9030 6000 30  0000 C CNN
+F 3 "~" H 9100 6000 30  0000 C CNN
+	1    9100 6000
+	0    -1   -1   0
+$EndComp
+$Comp
+L GND #PWR020
+U 1 1 552ABAF4
+P 9550 6000
+F 0 "#PWR020" H 9550 6000 30  0001 C CNN
+F 1 "GND" H 9550 5930 30  0001 C CNN
+F 2 "" H 9550 6000 60  0000 C CNN
+F 3 "" H 9550 6000 60  0000 C CNN
+	1    9550 6000
+	0    -1   -1   0
+$EndComp
+Wire Wire Line
+	9550 6000 9350 6000
+Wire Wire Line
+	8850 6000 7650 6000
+Wire Wire Line
+	7650 6000 7650 5700
+Wire Wire Line
+	4950 4800 5300 4800
+Connection ~ 5200 4900
+Wire Wire Line
+	2000 6350 3100 6350
+Wire Wire Line
+	3100 6350 3100 6800
+Wire Wire Line
+	3100 6800 4950 6800
+Wire Wire Line
+	4950 6800 4950 4800
+Connection ~ 5200 4800
+Connection ~ 2000 6350
 $EndSCHEMATC
