File: RS485-dry-contact.sch (KiCad schematic (older format))
At the start: 27 parts, among them IC1 ATMEGA168PA-A, IC2 SP3485EN, K1 CONN_3, P1 CONN_2, P2 CONN_6, P3 CONN_6, P4 CONN_2, P5 CONN_4, U1 7805, X1 CRYSTAL

Commit message: Добавлен список компонентов
Parts:
- C1: value CP1 -> 150uF 16V; footprint ~ -> c_tant_D
- C2: value C -> 0.01uF; footprint ~ -> SM1206
- C3: value C -> 0.1uf; footprint ~ -> SM1206
- C4, C5: value C -> 0.1uF; footprint ~ -> SM1206
- C7, C8: value C -> 22pF; footprint ~ -> SM1206
- D1, D3, D4, D5: footprint ~ -> LED-1206
- D2: footprint ~ -> PIN_ARRAY_4x1
- IC2: value SP3485EN -> MAX485CSA; footprint SO8 -> SO8N
- K1: footprint ~ -> bornier3
- P1, P4: footprint ~ -> bornier2
- P2, P3: footprint ~ -> PIN_ARRAY-6X1
- P5: footprint ~ -> bornier4
- R1, R3, R4, R5: value R -> 510; footprint ~ -> SM1206
- R2: value R -> 10k; footprint ~ -> SM1206
- U1: footprint ~ -> TO92
- X1: value CRYSTAL -> 16MHz; footprint ~ -> crystal_FA238-TSX3225
Connections:
- net GND: now also K1.1 (P1), K1.3 (P3), P5.3 (P3); no longer K1.2 (PM), P5.2 (P2), P5.4 (P4)
- net at C1.1, C2.2, D2.3 (+)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: now also K1.2 (PM); no longer P5.3 (P3)
- net at IC1.9 ((PCINT21/OC0B/T1)PD5): now also P5.4 (P4); no longer K1.1 (P1)
- no-connect marks 12 -> 13
Other:
- moved on the sheet: K1, P5
Changed lines of the file:
@@
 Sheet 1 1
 Title ""
-Date "12 apr 2015"
+Date "20 apr 2015"
 Rev ""
 Comp ""
@@
 F 0 "D2" H 2850 2200 70  0000 C CNN
 F 1 "BRIDGE" H 2850 2100 70  0000 C CNN
-F 2 "~" H 2850 2150 60  0000 C CNN
+F 2 "PIN_ARRAY_4x1" H 2850 2150 60  0000 C CNN
 F 3 "~" H 2850 2150 60  0000 C CNN
 	1    2850 2150
@@
 P 2900 3600
 F 0 "C1" H 2950 3700 50  0000 L CNN
-F 1 "CP1" H 2950 3500 50  0000 L CNN
-F 2 "~" H 2900 3600 60  0000 C CNN
+F 1 "150uF 16V" H 2950 3500 50  0000 L CNN
+F 2 "c_tant_D" H 2900 3600 60  0000 C CNN
 F 3 "~" H 2900 3600 60  0000 C CNN
 	1    2900 3600
@@
 P 2900 4150
 F 0 "C2" H 2900 4250 40  0000 L CNN
-F 1 "C" H 2906 4065 40  0000 L CNN
-F 2 "~" H 2938 4000 30  0000 C CNN
+F 1 "0.01uF" H 2906 4065 40  0000 L CNN
+F 2 "SM1206" H 2938 4000 30  0000 C CNN
 F 3 "~" H 2900 4150 60  0000 C CNN
 	1    2900 4150
@@
 F 0 "U1" H 3800 4854 60  0000 C CNN
 F 1 "7805" H 3650 5250 60  0000 C CNN
-F 2 "~" H 3650 5050 60  0000 C CNN
+F 2 "TO92" H 3650 5050 60  0000 C CNN
 F 3 "~" H 3650 5050 60  0000 C CNN
 	1    3650 5050
@@
 P 2900 5550
 F 0 "C3" H 2900 5650 40  0000 L CNN
-F 1 "C" H 2906 5465 40  0000 L CNN
-F 2 "~" H 2938 5400 30  0000 C CNN
+F 1 "0.1uf" H 2906 5465 40  0000 L CNN
+F 2 "SM1206" H 2938 5400 30  0000 C CNN
 F 3 "~" H 2900 5550 60  0000 C CNN
 	1    2900 5550
@@
 P 3200 5950
 F 0 "R1" V 3280 5950 40  0000 C CNN
-F 1 "R" V 3207 5951 40  0000 C CNN
-F 2 "~" V 3130 5950 30  0000 C CNN
+F 1 "510" V 3207 5951 40  0000 C CNN
+F 2 "SM1206" V 3130 5950 30  0000 C CNN
 F 3 "~" H 3200 5950 30  0000 C CNN
 	1    3200 5950
@@
 F 0 "D1" H 2400 6050 50  0000 C CNN
 F 1 "LED" H 2400 5850 50  0000 C CNN
-F 2 "~" H 2400 5950 60  0000 C CNN
+F 2 "LED-1206" H 2400 5950 60  0000 C CNN
 F 3 "~" H 2400 5950 60  0000 C CNN
 	1    2400 5950
@@
 F 0 "P1" V 700 2000 40  0000 C CNN
 F 1 "CONN_2" V 800 2000 40  0000 C CNN
-F 2 "~" H 750 2000 60  0000 C CNN
+F 2 "bornier2" H 750 2000 60  0000 C CNN
 F 3 "~" H 750 2000 60  0000 C CNN
 	1    750  2000
@@
 F 0 "P4" V 10750 4900 40  0000 C CNN
 F 1 "CONN_2" V 10850 4900 40  0000 C CNN
-F 2 "~" H 10800 4900 60  0000 C CNN
+F 2 "bornier2" H 10800 4900 60  0000 C CNN
 F 3 "~" H 10800 4900 60  0000 C CNN
 	1    10800 4900
@@
 P 5800 6150
 F 0 "C4" H 5800 6250 40  0000 L CNN
-F 1 "C" H 5806 6065 40  0000 L CNN
-F 2 "~" H 5838 6000 30  0000 C CNN
+F 1 "0.1uF" H 5806 6065 40  0000 L CNN
+F 2 "SM1206" H 5838 6000 30  0000 C CNN
 F 3 "~" H 5800 6150 60  0000 C CNN
 	1    5800 6150
@@
 P 6200 6150
 F 0 "C5" H 6200 6250 40  0000 L CNN
-F 1 "C" H 6206 6065 40  0000 L CNN
-F 2 "~" H 6238 6000 30  0000 C CNN
+F 1 "0.1uF" H 6206 6065 40  0000 L CNN
+F 2 "SM1206" H 6238 6000 30  0000 C CNN
 F 3 "~" H 6200 6150 60  0000 C CNN
 	1    6200 6150
@@
 F 0 "P2" V 10750 2900 60  0000 C CNN
 F 1 "CONN_6" V 10850 2900 60  0000 C CNN
-F 2 "~" H 10800 2900 60  0000 C CNN
+F 2 "PIN_ARRAY-6X1" H 10800 2900 60  0000 C CNN
 F 3 "~" H 10800 2900 60  0000 C CNN
 	1    10800 2900
@@
 P 7750 2200
 F 0 "X1" H 7750 2350 60  0000 C CNN
-F 1 "CRYSTAL" H 7750 2050 60  0000 C CNN
-F 2 "~" H 7750 2200 60  0000 C CNN
+F 1 "16MHz" H 7750 2050 60  0000 C CNN
+F 2 "crystal_FA238-TSX3225" H 7750 2200 60  0000 C CNN
 F 3 "~" H 7750 2200 60  0000 C CNN
 	1    7750 2200
@@
 P 7450 1750
 F 0 "C7" H 7450 1850 40  0000 L CNN
-F 1 "C" H 7456 1665 40  0000 L CNN
-F 2 "~" H 7488 1600 30  0000 C CNN
+F 1 "22pF" H 7456 1665 40  0000 L CNN
+F 2 "SM1206" H 7488 1600 30  0000 C CNN
 F 3 "~" H 7450 1750 60  0000 C CNN
 	1    7450 1750
@@
 P 8050 1750
 F 0 "C8" H 8050 1850 40  0000 L CNN
-F 1 "C" H 8056 1665 40  0000 L CNN
-F 2 "~" H 8088 1600 30  0000 C CNN
+F 1 "22pF" H 8056 1665 40  0000 L CNN
+F 2 "SM1206" H 8088 1600 30  0000 C CNN
 F 3 "~" H 8050 1750 60  0000 C CNN
 	1    8050 1750
@@
 P 8950 4900
 F 0 "IC2" H 8750 5150 40  0000 C CNN
-F 1 "SP3485EN" H 9150 4650 40  0000 C CNN
-F 2 "SO8" H 8950 4900 35  0000 C CIN
+F 1 "MAX485CSA" H 9150 4650 40  0000 C CNN
+F 2 "SO8N" H 8950 4900 35  0000 C CIN
 F 3 "" H 8950 4900 60  0000 C CNN
 	1    8950 4900
@@
 	3700 2150 3700 4650
 Wire Wire Line
-	3100 3600 4650 3600
+	4650 3600 3100 3600
 Wire Wire Line
 	2000 2150 2000 6500
@@
 	7200 4800 7300 4800
 Wire Wire Line
-	4450 1750 4450 5350
+	4450 1650 4450 5350
 Wire Wire Line
 	4450 5350 7550 5350
@@
 $EndComp
 Wire Wire Line
-	4250 2000 4250 1750
+	4250 1550 4250 2000
 $Comp
 L GND #PWR015
@@
 $EndComp
 Wire Wire Line
-	4550 2000 4550 1750
-Wire Wire Line
-	4650 3600 4650 1750
+	4550 1200 4550 2000
+Wire Wire Line
+	4650 1300 4650 3600
 $Comp
 L GND #PWR016
@@
 $EndComp
 Wire Wire Line
-	4750 2000 4750 1750
+	4750 1500 4750 2000
 $Comp
 L CONN_6 P3
@@
 F 0 "P3" V 9450 2900 60  0000 C CNN
 F 1 "CONN_6" V 9550 2900 60  0000 C CNN
-F 2 "~" H 9500 2900 60  0000 C CNN
+F 2 "PIN_ARRAY-6X1" H 9500 2900 60  0000 C CNN
 F 3 "~" H 9500 2900 60  0000 C CNN
 	1    9500 2900
@@
 P 9050 3900
 F 0 "R2" V 9130 3900 40  0000 C CNN
-F 1 "R" V 9057 3901 40  0000 C CNN
-F 2 "~" V 8980 3900 30  0000 C CNN
+F 1 "10k" V 9057 3901 40  0000 C CNN
+F 2 "SM1206" V 8980 3900 30  0000 C CNN
 F 3 "~" H 9050 3900 30  0000 C CNN
 	1    9050 3900
@@
 	8050 4850 8550 4850
 Wire Wire Line
-	4150 1750 4150 2200
+	4150 1400 4150 2200
 Wire Wire Line
 	4150 2200 7300 2200
@@
 L CONN_3 K1
 U 1 1 552AB124
-P 4250 1400
-F 0 "K1" V 4200 1400 50  0000 C CNN
-F 1 "CONN_3" V 4300 1400 40  0000 C CNN
-F 2 "~" H 4250 1400 60  0000 C CNN
-F 3 "~" H 4250 1400 60  0000 C CNN
-	1    4250 1400
+P 4100 750
+F 0 "K1" V 4050 750 50  0000 C CNN
+F 1 "CONN_3" V 4150 750 40  0000 C CNN
+F 2 "bornier3" H 4100 750 60  0000 C CNN
+F 3 "~" H 4100 750 60  0000 C CNN
+	1    4100 750
 	0    -1   -1   0
 $EndComp
@@
 L CONN_4 P5
 U 1 1 552AB135
-P 4600 1400
-F 0 "P5" V 4550 1400 50  0000 C CNN
-F 1 "CONN_4" V 4650 1400 50  0000 C CNN
-F 2 "~" H 4600 1400 60  0000 C CNN
-F 3 "~" H 4600 1400 60  0000 C CNN
-	1    4600 1400
+P 5300 650
+F 0 "P5" V 5250 650 50  0000 C CNN
+F 1 "CONN_4" V 5350 650 50  0000 C CNN
+F 2 "bornier4" H 5300 650 60  0000 C CNN
+F 3 "~" H 5300 650 60  0000 C CNN
+	1    5300 650
 	0    -1   -1   0
 $EndComp
@@
 F 0 "D3" H 8500 4550 50  0000 C CNN
 F 1 "LED" H 8500 4350 50  0000 C CNN
-F 2 "~" H 8500 4450 60  0000 C CNN
+F 2 "LED-1206" H 8500 4450 60  0000 C CNN
 F 3 "~" H 8500 4450 60  0000 C CNN
 	1    8500 4450
@@
 P 9050 4100
 F 0 "R3" V 9130 4100 40  0000 C CNN
-F 1 "R" V 9057 4101 40  0000 C CNN
-F 2 "~" V 8980 4100 30  0000 C CNN
+F 1 "510" V 9057 4101 40  0000 C CNN
+F 2 "SM1206" V 8980 4100 30  0000 C CNN
 F 3 "~" H 9050 4100 30  0000 C CNN
 	1    9050 4100
@@
 F 0 "D4" H 8500 5600 50  0000 C CNN
 F 1 "LED" H 8500 5400 50  0000 C CNN
-F 2 "~" H 8500 5500 60  0000 C CNN
+F 2 "LED-1206" H 8500 5500 60  0000 C CNN
 F 3 "~" H 8500 5500 60  0000 C CNN
 	1    8500 5500
@@
 P 9100 5800
 F 0 "R4" V 9180 5800 40  0000 C CNN
-F 1 "R" V 9107 5801 40  0000 C CNN
-F 2 "~" V 9030 5800 30  0000 C CNN
+F 1 "510" V 9107 5801 40  0000 C CNN
+F 2 "SM1206" V 9030 5800 30  0000 C CNN
 F 3 "~" H 9100 5800 30  0000 C CNN
 	1    9100 5800
@@
 F 0 "D5" H 7650 5600 50  0000 C CNN
 F 1 "LED" H 7650 5400 50  0000 C CNN
-F 2 "~" H 7650 5500 60  0000 C CNN
+F 2 "LED-1206" H 7650 5500 60  0000 C CNN
 F 3 "~" H 7650 5500 60  0000 C CNN
 	1    7650 5500
@@
 P 9100 6000
 F 0 "R5" V 9180 6000 40  0000 C CNN
-F 1 "R" V 9107 6001 40  0000 C CNN
-F 2 "~" V 9030 6000 30  0000 C CNN
+F 1 "510" V 9107 6001 40  0000 C CNN
+F 2 "SM1206" V 9030 6000 30  0000 C CNN
 F 3 "~" H 9100 6000 30  0000 C CNN
 	1    9100 6000
@@
 Connection ~ 5200 4800
 Connection ~ 2000 6350
+Wire Wire Line
+	4150 1400 5450 1400
+Wire Wire Line
+	5450 1400 5450 1000
+Wire Wire Line
+	4250 1550 5350 1550
+Wire Wire Line
+	5350 1550 5350 1000
+Wire Wire Line
+	4450 1650 5150 1650
+Wire Wire Line
+	5150 1650 5150 1000
+Wire Wire Line
+	4550 1200 4200 1200
+Wire Wire Line
+	4200 1200 4200 1100
+Wire Wire Line
+	4650 1300 4100 1300
+Wire Wire Line
+	4100 1300 4100 1100
+Wire Wire Line
+	4750 1500 4000 1500
+Wire Wire Line
+	4000 1500 4000 1100
+NoConn ~ 5250 1000
 $EndSCHEMATC
